Commit message: cleaned up packages that were un-needed for now. Can fold them back in as needed

File: rover_desc_pkg/urdf/links_joints.xacro (robot description, xacro)
@@ -1,4 +1,7 @@
 <?xml version="1.0"?>
 <robot xmlns:xacro="http://www.ros.org/wiki/xacro">
+  <!-- Begin - Include -->
+    <xacro:include filename="$(find rover_desc_pkg)/urdf/common_materials.xacro"/>
+  <!-- End - Include -->
   <!-- Joint Macro -->
   <!-- fixed joint -->
@@ -12,5 +15,6 @@
   </xacro:macro>
   <!-- continuous joint -->
-  <xacro:macro name="m_joint_cont" params="name axis_xyz origin_xyz origin_rpy parent child limit_e limit_v">
+  <xacro:macro name="m_joint_cont" params="name axis_xyz origin_xyz origin_rpy
+               parent child limit_e limit_v damp fric">
     <joint name="${name}" type="continuous">
       <axis xyz="${axis_xyz}"/>
@@ -19,4 +23,5 @@
       <parent link="${parent}"/>
       <child link="${child}"/>
+      <dynamics damping="${damp}" friction="${fric}"/>
     </joint>
     <transmission name="trans_${name}">
@@ -32,11 +37,14 @@
   </xacro:macro>
   <!-- revolute joint -->
-  <xacro:macro name="m_joint_rev" params="name axis_xyz origin_xyz origin_rpy parent child limit_e limit_l limit_u limit_v">
+  <xacro:macro name="m_joint_rev" params="name axis_xyz axis_rpy origin_xyz
+               origin_rpy parent child limit_e limit_l limit_u limit_v damp
+               fric">
     <joint name="${name}" type="revolute">
-      <axis xyz="${axis_xyz}"/>
+      <axis rpy="axis_rpy" xyz="${axis_xyz}"/>
       <limit effort="${limit_e}" lower="${limit_l}" upper="${limit_u}" velocity="${limit_v}"/>
       <origin rpy="${origin_rpy}" xyz="${origin_xyz}"/>
       <parent link="${parent}"/>
       <child link="${child}"/>
+      <dynamics damping="${damp}" friction="${fric}"/>
     </joint>
     <transmission name="trans_${name}">
@@ -51,16 +59,30 @@
     </transmission>
   </xacro:macro>
-  <!-- Cylinder link Macro -->
-  <xacro:macro name="m_link_cylinder" params="name color origin_xyz origin_rpy radius length mass ixx ixy ixz iyy iyz izz">
+  <!-- Cylinder link Macro without inertia -->
+  <xacro:macro name="m_link_cylinder" params="name origin_xyz origin_rpy r l">
+    <link name="${name}">
+      <visual>
+        <origin rpy="${origin_rpy}" xyz="${origin_xyz}"/>
+        <geometry>
+          <cylinder radius="${r}" length="${l}"/>
+        </geometry>
+        <xacro:material_gray/>
+      </visual>
+    </link>
+  </xacro:macro>
+  <!-- Cylinder link Macro with inertia -->
+  <xacro:macro name="m_link_cylinder_inertia" params="name origin_xyz origin_rpy r l m">
     <link name="${name}">
       <inertial>
-        <mass value="${mass}"/>
+        <mass value="${m}"/>
         <origin rpy="${origin_rpy}" xyz="${origin_xyz}"/>
-        <inertia ixx="${ixx}" ixy="${ixy}" ixz="${ixz}" iyy="${iyy}" iyz="${iyz}" izz="${izz}"/>
+        <inertia ixx="${m*(3*r*r+l*l)/12}" ixy="0.0" ixz="0.0"
+                 iyy="${m*(3*r*r+l*l)/12}" iyz="0.0"
+                 izz="${m*r*r/2}"/>
       </inertial>
       <collision>
         <origin rpy="${origin_rpy}" xyz="${origin_xyz}"/>
         <geometry>
-          <cylinder radius="${radius}" length="${length}"/>
+          <cylinder radius="${r}" length="${l}"/>
         </geometry>
       </collision>
@@ -68,24 +90,36 @@
         <origin rpy="${origin_rpy}" xyz="${origin_xyz}"/>
         <geometry>
-          <cylinder radius="${radius}" length="${length}"/>
+          <cylinder radius="${r}" length="${l}"/>
         </geometry>
-        <material name="">
-          <color rgba="${color}"/>
-        </material>
+        <xacro:material_darkgray/>
       </visual>
     </link>
   </xacro:macro>
-  <!-- Box link Macro -->
-  <xacro:macro name="m_link_box" params="name color origin_xyz origin_rpy size mass ixx ixy ixz iyy iyz izz">
+  <!-- Box link Macro without inertia -->
+  <xacro:macro name="m_link_box" params="name origin_xyz origin_rpy w d h">
+    <link name="${name}">
+      <visual>
+        <origin rpy="${origin_rpy}" xyz="${origin_xyz}"/>
+        <geometry>
+          <box size="${w} ${d} ${h}"/>
+        </geometry>
+        <xacro:material_white/>
+      </visual>
+    </link>
+  </xacro:macro>
+  <!-- Box link Macro with inertia -->
+  <xacro:macro name="m_link_box_inertia" params="name origin_xyz origin_rpy m w d h">
     <link name="${name}">
       <inertial>
-        <mass value="${mass}"/>
+        <mass value="${m}"/>
         <origin rpy="${origin_rpy}" xyz="${origin_xyz}"/>
-        <inertia ixx="${ixx}" ixy="${ixy}" ixz="${ixz}" iyy="${iyy}" iyz="${iyz}" izz="${izz}"/>
+        <inertia ixx="${m*(d*d+h*h)/12}" ixy="0" ixz="0"
+                 iyy="${m*(w*w+h*h)/12}" iyz="0"
+                 izz="${m*(w*w+d*d)/12}"/>
       </inertial>
       <collision>
         <origin rpy="${origin_rpy}" xyz="${origin_xyz}"/>
         <geometry>
-          <box size="${size}"/>
+          <box size="${w} ${d} ${h}"/>
         </geometry>
       </collision>
@@ -93,19 +127,19 @@
         <origin rpy="${origin_rpy}" xyz="${origin_xyz}"/>
         <geometry>
-          <box size="${size}"/>
+          <box size="${w} ${d} ${h}"/>
         </geometry>
-        <material name="">
-          <color rgba="${color}"/>
-        </material>
+        <xacro:material_clay_brown/>
       </visual>
     </link>
   </xacro:macro>
-  <!-- Mesh link Macro -->
-  <xacro:macro name="m_link_mesh" params="name color origin_xyz origin_rpy meshfile meshscale mass ixx ixy ixz iyy iyz izz">
+  <!-- Mesh link Macro Box -->
+  <xacro:macro name="m_link_mesh_box" params="name origin_xyz origin_rpy meshfile meshscale m w d h">
     <link name="${name}">
       <inertial>
-        <mass value="${mass}"/>
+        <mass value="${m}"/>
         <origin rpy="${origin_rpy}" xyz="${origin_xyz}"/>
-        <inertia ixx="${ixx}" ixy="${ixy}" ixz="${ixz}" iyy="${iyy}" iyz="${iyz}" izz="${izz}"/>
+        <inertia ixx="${m*(d*d+h*h)/12}" ixy="0" ixz="0"
+                 iyy="${m*(w*w+h*h)/12}" iyz="0"
+                 izz="${m*(w*w+d*d)/12}"/>
       </inertial>
       <collision>
@@ -120,7 +154,28 @@
             <mesh filename="${meshfile}" scale="${meshscale}"/>
         </geometry>
-        <material name="">
-            <color rgba="${color}"/>
-        </material>
+      </visual>
+    </link>
+  </xacro:macro>
+  <!-- Mesh link Macro Cylinder -->
+  <xacro:macro name="m_link_mesh_cyl" params="name origin_xyz origin_rpy meshfile meshscale m r l">
+    <link name="${name}">
+      <inertial>
+        <mass value="${m}"/>
+        <origin rpy="${origin_rpy}" xyz="${origin_xyz}"/>
+        <inertia ixx="${m*(3*r*l+r*l)/12}" ixy="0.0" ixz="0.0"
+                 iyy="${m*(3*r*r+l*l)/12}" iyz="0.0"
+                 izz="${m*l*l/2}"/>
+      </inertial>
+      <collision>
+        <origin rpy="${origin_rpy}" xyz="${origin_xyz}"/>
+        <geometry>
+            <mesh filename="${meshfile}" scale="${meshscale}"/>
+        </geometry>
+      </collision>
+      <visual>
+        <origin rpy="${origin_rpy}" xyz="${origin_xyz}"/>
+        <geometry>
+            <mesh filename="${meshfile}" scale="${meshscale}"/>
+        </geometry>
       </visual>
     </link>
